Commit message: ~90% computation Package

File: src/sparsh_computation/urdf/sparsh.xacro (robot description, xacro)
@@ -156,5 +156,5 @@
   </link>
   <!-- BOTTOM LEFT COLUMN LINK-->
-    <link name="column_link_bottom_left">
+  <link name="column_link_bottom_left">
     <visual>
       <origin xyz="0 0 ${column_height/2}" rpy="0 0 0"/>
@@ -179,5 +179,5 @@
       <child link="column_link_top_right"/>
   </joint>
-    <joint name="top_left_column_to_base_link" type="prismatic">
+  <joint name="top_left_column_to_base_link" type="prismatic">
       <origin xyz="-${spacing_x} -${spacing_y} ${base_height}" rpy="0 0 0"/>
       <limit upper="${upper_limit}" lower="0" effort="500" velocity="${vel}"/>
@@ -186,5 +186,5 @@
       <child link="column_link_top_left"/>
   </joint>
-    <joint name="middle_right_column_to_base_link" type="prismatic">
+  <joint name="middle_right_column_to_base_link" type="prismatic">
       <origin xyz="0 ${spacing_y} ${base_height}" rpy="0 0 0"/>
       <limit upper="${upper_limit}" lower="0" effort="500" velocity="${vel}"/>
@@ -193,5 +193,5 @@
       <child link="column_link_middle_right"/>
   </joint>
-    <joint name="middle_left_column_to_base_link" type="prismatic">
+  <joint name="middle_left_column_to_base_link" type="prismatic">
       <origin xyz="0 -${spacing_y} ${base_height}" rpy="0 0 0"/>
       <limit upper="${upper_limit}" lower="0" effort="500" velocity="${vel}"/>
@@ -200,5 +200,5 @@
       <child link="column_link_middle_left"/>
   </joint>
-    <joint name="bottom_right_column_to_base_link" type="prismatic">
+  <joint name="bottom_right_column_to_base_link" type="prismatic">
       <origin xyz="${spacing_x} ${spacing_y} ${base_height}" rpy="0 0 0"/>
       <limit upper="${upper_limit}" lower="0" effort="500" velocity="${vel}"/>
@@ -207,5 +207,5 @@
       <child link="column_link_bottom_right"/>
   </joint>
-    <joint name="bottom_left_column_to_base_link" type="prismatic">
+  <joint name="bottom_left_column_to_base_link" type="prismatic">
       <origin xyz="${spacing_x} -${spacing_y} ${base_height}" rpy="0 0 0"/>
       <limit upper="${upper_limit}" lower="0" effort="500" velocity="${vel}"/>
@@ -214,70 +214,3 @@
       <child link="column_link_bottom_left"/>
   </joint>
-  <!-- TRANSMISSION INTERFACE -->
-  <transmission name="top_right_column_to_base">
-    <type>transmission_interface/SimpleTransmission</type>
-    <joint name="top_right_column_to_base_link">
-      <hardwareInterface>hardware_interface/EffortJointInterface</hardwareInterface>
-    </joint>
-    <actuator name="top_right_column_to_base_actuator">
-      <hardwareInterface>hardware_interface/EffortJointInterface</hardwareInterface>
-      <mechanicalReduction>1</mechanicalReduction>
-    </actuator>
-  </transmission>
-  <transmission name="top_left_column_to_base">
-    <type>transmission_interface/SimpleTransmission</type>
-    <joint name="top_left_column_to_base_link">
-      <hardwareInterface>hardware_interface/EffortJointInterface</hardwareInterface>
-    </joint>
-    <actuator name="top_left_column_to_base_actuator">
-      <hardwareInterface>hardware_interface/EffortJointInterface</hardwareInterface>
-      <mechanicalReduction>1</mechanicalReduction>
-    </actuator>
-  </transmission>
-  <transmission name="middle_right_column_to_base">
-    <type>transmission_interface/SimpleTransmission</type>
-    <joint name="middle_right_column_to_base_link">
-      <hardwareInterface>hardware_interface/EffortJointInterface</hardwareInterface>
-    </joint>
-    <actuator name="middle_right_column_to_base_actuator">
-      <hardwareInterface>hardware_interface/EffortJointInterface</hardwareInterface>
-      <mechanicalReduction>1</mechanicalReduction>
-    </actuator>
-  </transmission>
-  <transmission name="middle_left_column_to_base">
-    <type>transmission_interface/SimpleTransmission</type>
-    <joint name="middle_left_column_to_base_link">
-      <hardwareInterface>hardware_interface/EffortJointInterface</hardwareInterface>
-    </joint>
-    <actuator name="middle_left_column_to_base_actuator">
-      <hardwareInterface>hardware_interface/EffortJointInterface</hardwareInterface>
-      <mechanicalReduction>1</mechanicalReduction>
-    </actuator>
-  </transmission>
-  <transmission name="bottom_right_column_to_base">
-    <type>transmission_interface/SimpleTransmission</type>
-    <joint name="bottom_right_column_to_base_link">
-      <hardwareInterface>hardware_interface/EffortJointInterface</hardwareInterface>
-    </joint>
-    <actuator name="bottom_right_column_to_base_actuator">
-      <hardwareInterface>hardware_interface/EffortJointInterface</hardwareInterface>
-      <mechanicalReduction>1</mechanicalReduction>
-    </actuator>
-  </transmission>
-  <transmission name="bottom_left_column_to_base">
-    <type>transmission_interface/SimpleTransmission</type>
-    <joint name="bottom_left_column_to_base_link">
-      <hardwareInterface>hardware_interface/EffortJointInterface</hardwareInterface>
-    </joint>
-    <actuator name="bottom_left_column_to_base_actuator">
-      <hardwareInterface>hardware_interface/EffortJointInterface</hardwareInterface>
-      <mechanicalReduction>1</mechanicalReduction>
-    </actuator>
-  </transmission>
-  <gazebo>
-    <plugin name="gazebo_ros_control" filename="libgazebo_ros_control.so">
-      <robotNamespace>/sparsh</robotNamespace>
-      <robotSimType>gazebo_ros_control/DefaultRobotHWSim</robotSimType>
-    </plugin>
-  </gazebo>
 </robot>

File: src/sparsh_computation/urdf/sparsh_plugins.xacro (robot description, xacro)
@@ -1,3 +1,72 @@
 <?xml version="1.0"?>
-<robot>
+<robot name="sparsh" xmlns:xacro="http://ros.org/wiki/xacro"
+            xmlns:sensor="http://playerstage.sourceforge.net/gazebo/xmlschema/#sensor"
+            xmlns:controller="http://playerstage.sourceforge.net/gazebo/xmlschema/#controller"
+            xmlns:interface="http://playerstage.sourceforge.net/gazebo/xmlschema/#interface">
+  <transmission name="top_right_column_to_base">
+    <type>transmission_interface/SimpleTransmission</type>
+    <joint name="top_right_column_to_base_link">
+      <hardwareInterface>hardware_interface/EffortJointInterface</hardwareInterface>
+    </joint>
+    <actuator name="top_right_column_to_base_actuator">
+      <hardwareInterface>hardware_interface/EffortJointInterface</hardwareInterface>
+      <mechanicalReduction>1</mechanicalReduction>
+    </actuator>
+  </transmission>
+  <transmission name="top_left_column_to_base">
+    <type>transmission_interface/SimpleTransmission</type>
+    <joint name="top_left_column_to_base_link">
+      <hardwareInterface>hardware_interface/EffortJointInterface</hardwareInterface>
+    </joint>
+    <actuator name="top_left_column_to_base_actuator">
+      <hardwareInterface>hardware_interface/EffortJointInterface</hardwareInterface>
+      <mechanicalReduction>1</mechanicalReduction>
+    </actuator>
+  </transmission>
+  <transmission name="middle_right_column_to_base">
+    <type>transmission_interface/SimpleTransmission</type>
+    <joint name="middle_right_column_to_base_link">
+      <hardwareInterface>hardware_interface/EffortJointInterface</hardwareInterface>
+    </joint>
+    <actuator name="middle_right_column_to_base_actuator">
+      <hardwareInterface>hardware_interface/EffortJointInterface</hardwareInterface>
+      <mechanicalReduction>1</mechanicalReduction>
+    </actuator>
+  </transmission>
+  <transmission name="middle_left_column_to_base">
+    <type>transmission_interface/SimpleTransmission</type>
+    <joint name="middle_left_column_to_base_link">
+      <hardwareInterface>hardware_interface/EffortJointInterface</hardwareInterface>
+    </joint>
+    <actuator name="middle_left_column_to_base_actuator">
+      <hardwareInterface>hardware_interface/EffortJointInterface</hardwareInterface>
+      <mechanicalReduction>1</mechanicalReduction>
+    </actuator>
+  </transmission>
+  <transmission name="bottom_right_column_to_base">
+    <type>transmission_interface/SimpleTransmission</type>
+    <joint name="bottom_right_column_to_base_link">
+      <hardwareInterface>hardware_interface/EffortJointInterface</hardwareInterface>
+    </joint>
+    <actuator name="bottom_right_column_to_base_actuator">
+      <hardwareInterface>hardware_interface/EffortJointInterface</hardwareInterface>
+      <mechanicalReduction>1</mechanicalReduction>
+    </actuator>
+  </transmission>
+  <transmission name="bottom_left_column_to_base">
+    <type>transmission_interface/SimpleTransmission</type>
+    <joint name="bottom_left_column_to_base_link">
+      <hardwareInterface>hardware_interface/EffortJointInterface</hardwareInterface>
+    </joint>
+    <actuator name="bottom_left_column_to_base_actuator">
+      <hardwareInterface>hardware_interface/EffortJointInterface</hardwareInterface>
+      <mechanicalReduction>1</mechanicalReduction>
+    </actuator>
+  </transmission>
+  <gazebo>
+    <plugin name="gazebo_ros_control" filename="libgazebo_ros_control.so">
+      <robotNamespace>/sparsh</robotNamespace>
+      <robotSimType>gazebo_ros_control/DefaultRobotHWSim</robotSimType>
+    </plugin>
+  </gazebo>
 </robot>

Commit message: update scroll_pos in yaml updated gio

File: src/sparsh_computation/urdf/sparsh.xacro (robot description, xacro)
@@ -23,5 +23,5 @@
   <xacro:property name="spacing_y" value="0.05"/>
   <xacro:property name="upper_limit" value="0.1"/>
-  <xacro:property name="vel" value="0.1"/>
+  <xacro:property name="vel" value="30"/>
   <!-- COLOURS FOR MATERIAL -->
   <material name="white">
